File: Esquemático acionamento/Esquemático.sch (EAGLE design)
At the start: 9 parts, among them Q1 IRF540, Q2 IRF540

Commit message: Add files via upload
Placa de Acionamento
Parts:
- removed Q1: IRF540, transistor-fet:IRF540
- removed R2: 1k, rcl:R-EU_0204/7
- removed U$3: JST2.54X2P, CRD:JST2.54X2P
Connections:
- removed net N$3: Q1.G, R2.2, U$3.1
- removed net N$5: Q1.D, SP1.1
- net 0: now also SP1.1; no longer Q1.S, R2.1
- net N$1: now also SP1.2
- net VCC: no longer SP1.2
Other:
- moved on the sheet: SP1
Changed lines of the file:
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@@
 <drawing>
 <settings>
-<setting alwaysvectorfont="yes"/>
+<setting alwaysvectorfont="no"/>
 <setting verticaltext="up"/>
 </settings>
-<grid distance="0.1" unitdist="inch" unit="inch" style="lines" multiple="1" display="no" altdistance="0.01" altunitdist="inch" altunit="inch"/>
+<grid distance="0.1" unitdist="inch" unit="mil" style="lines" multiple="1" display="yes" altdistance="0.01" altunitdist="inch" altunit="inch"/>
 <layers>
 <layer number="1" name="Top" color="4" fill="1" visible="no" active="no"/>
@@
 <parts>
 <part name="FRAME1" library="frames" library_urn="urn:adsk.eagle:library:229" deviceset="A4L-LOC" device=""/>
-<part name="Q1" library="transistor-fet" library_urn="urn:adsk.eagle:library:396" deviceset="IRF540" device="" package3d_urn="urn:adsk.eagle:package:28520/1"/>
 <part name="U$1" library="CRD" library_urn="urn:adsk.eagle:library:39051337" deviceset="JST2.54X2P" device="" package3d_urn="urn:adsk.eagle:package:39191967/2"/>
 <part name="U$2" library="CRD" library_urn="urn:adsk.eagle:library:39051337" deviceset="JST2.54X2P" device="" package3d_urn="urn:adsk.eagle:package:39191967/2"/>
 <part name="R1" library="rcl" library_urn="urn:adsk.eagle:library:334" deviceset="R-EU_" device="0204/7" package3d_urn="urn:adsk.eagle:package:23498/2" value="1k"/>
 <part name="Q2" library="transistor-fet" library_urn="urn:adsk.eagle:library:396" deviceset="IRF540" device="" package3d_urn="urn:adsk.eagle:package:28520/1"/>
-<part name="R2" library="rcl" library_urn="urn:adsk.eagle:library:334" deviceset="R-EU_" device="0204/7" package3d_urn="urn:adsk.eagle:package:23498/2" value="1k"/>
 <part name="X_1" library="ngspice-simulation" library_urn="urn:adsk.eagle:library:527439" deviceset="GND" device=""/>
 <part name="X_2" library="ngspice-simulation" library_urn="urn:adsk.eagle:library:527439" deviceset="GND" device=""/>
 <part name="X_3" library="ngspice-simulation" library_urn="urn:adsk.eagle:library:527439" deviceset="GND" device=""/>
-<part name="U$3" library="CRD" library_urn="urn:adsk.eagle:library:39051337" deviceset="JST2.54X2P" device="" package3d_urn="urn:adsk.eagle:package:39191967/2"/>
 <part name="P+1" library="supply1" library_urn="urn:adsk.eagle:library:371" deviceset="VCC" device=""/>
-<part name="X_5" library="ngspice-simulation" library_urn="urn:adsk.eagle:library:527439" deviceset="GND" device=""/>
-<part name="P+2" library="supply1" library_urn="urn:adsk.eagle:library:371" deviceset="VCC" device=""/>
 <part name="P+3" library="supply1" library_urn="urn:adsk.eagle:library:371" deviceset="VCC" device=""/>
 <part name="X_4" library="ngspice-simulation" library_urn="urn:adsk.eagle:library:527439" deviceset="GND" device=""/>
@@
 <attribute name="SHEET" x="108.585" y="-81.28" size="2.54" layer="94"/>
 </instance>
-<instance part="Q1" gate="G$1" x="93.98" y="30.48" smashed="yes" rot="MR0">
-<attribute name="VALUE" x="105.41" y="30.48" size="1.778" layer="96" rot="MR0"/>
-<attribute name="NAME" x="105.41" y="33.02" size="1.778" layer="95" rot="MR0"/>
-</instance>
 <instance part="U$1" gate="G$1" x="124.46" y="-15.24" smashed="yes" rot="MR90"/>
 <instance part="U$2" gate="G$1" x="73.66" y="-7.62" smashed="yes" rot="MR270"/>
@@
 <attribute name="NAME" x="105.41" y="-20.32" size="1.778" layer="95" rot="MR0"/>
 </instance>
-<instance part="R2" gate="G$1" x="106.68" y="22.86" smashed="yes" rot="R90">
-<attribute name="NAME" x="105.1814" y="19.05" size="1.778" layer="95" rot="R90"/>
-<attribute name="VALUE" x="109.982" y="19.05" size="1.778" layer="96" rot="R90"/>
-</instance>
 <instance part="X_1" gate="G$1" x="88.9" y="-40.64" smashed="yes"/>
-<instance part="X_2" gate="G$1" x="106.68" y="12.7" smashed="yes"/>
+<instance part="X_2" gate="G$1" x="111.76" y="17.78" smashed="yes" rot="MR180"/>
 <instance part="X_3" gate="G$1" x="111.76" y="-40.64" smashed="yes" rot="MR0"/>
-<instance part="U$3" gate="G$1" x="124.46" y="38.1" smashed="yes" rot="MR90"/>
 <instance part="P+1" gate="VCC" x="88.9" y="5.08" smashed="yes">
 <attribute name="VALUE" x="86.36" y="2.54" size="1.778" layer="96" rot="R90"/>
-</instance>
-<instance part="X_5" gate="G$1" x="88.9" y="12.7" smashed="yes"/>
-<instance part="P+2" gate="VCC" x="81.28" y="50.8" smashed="yes">
-<attribute name="VALUE" x="78.74" y="48.26" size="1.778" layer="96" rot="R90"/>
 </instance>
 <instance part="P+3" gate="VCC" x="60.96" y="27.94" smashed="yes">
@@
 </instance>
 <instance part="X_4" gate="G$1" x="60.96" y="5.08" smashed="yes"/>
-<instance part="SP1" gate="G$1" x="81.28" y="35.56" smashed="yes" rot="R90">
-<attribute name="NAME" x="74.93" y="31.75" size="1.778" layer="95" rot="R90"/>
-<attribute name="VALUE" x="84.455" y="31.75" size="1.778" layer="96" rot="R90"/>
+<instance part="SP1" gate="G$1" x="111.76" y="7.62" smashed="yes" rot="MR270">
+<attribute name="NAME" x="105.41" y="11.43" size="1.778" layer="95" rot="MR270"/>
+<attribute name="VALUE" x="114.935" y="11.43" size="1.778" layer="96" rot="MR270"/>
 </instance>
 <instance part="U$4" gate="G$1" x="48.26" y="15.24" smashed="yes" rot="MR270"/>
@@
 </segment>
 <segment>
-<pinref part="R2" gate="G$1" pin="1"/>
-<pinref part="X_2" gate="G$1" pin="0"/>
-<wire x1="106.68" y1="17.78" x2="106.68" y2="12.7" width="0.1524" layer="91"/>
-</segment>
-<segment>
-<pinref part="X_5" gate="G$1" pin="0"/>
-<pinref part="Q1" gate="G$1" pin="S"/>
-<wire x1="88.9" y1="12.7" x2="88.9" y2="27.94" width="0.1524" layer="91"/>
-</segment>
-<segment>
 <pinref part="X_4" gate="G$1" pin="0"/>
 <wire x1="60.96" y1="12.7" x2="60.96" y2="5.08" width="0.1524" layer="91"/>
 <pinref part="U$4" gate="G$1" pin="2"/>
 <wire x1="58.42" y1="12.7" x2="60.96" y2="12.7" width="0.1524" layer="91"/>
+</segment>
+<segment>
+<pinref part="SP1" gate="G$1" pin="1"/>
+<pinref part="X_2" gate="G$1" pin="0"/>
+<wire x1="111.76" y1="12.7" x2="111.76" y2="17.78" width="0.1524" layer="91"/>
 </segment>
 </net>
@@
 <junction x="111.76" y="-25.4"/>
 <pinref part="Q2" gate="G$1" pin="G"/>
+<pinref part="SP1" gate="G$1" pin="2"/>
+<wire x1="111.76" y1="-17.78" x2="111.76" y2="2.54" width="0.1524" layer="91"/>
+<junction x="111.76" y="-17.78"/>
 </segment>
 </net>
@@
 </segment>
 </net>
-<net name="N$3" class="0">
-<segment>
-<pinref part="R2" gate="G$1" pin="2"/>
-<wire x1="106.68" y1="27.94" x2="114.3" y2="27.94" width="0.1524" layer="91"/>
-<pinref part="U$3" gate="G$1" pin="1"/>
-<wire x1="114.3" y1="27.94" x2="114.3" y2="35.56" width="0.1524" layer="91"/>
-<pinref part="Q1" gate="G$1" pin="G"/>
-<wire x1="106.68" y1="27.94" x2="99.06" y2="27.94" width="0.1524" layer="91"/>
-<junction x="106.68" y="27.94"/>
-</segment>
-</net>
 <net name="VCC" class="0">
-<segment>
-<pinref part="P+2" gate="VCC" pin="VCC"/>
-<wire x1="81.28" y1="48.26" x2="81.28" y2="40.64" width="0.1524" layer="91"/>
-<pinref part="SP1" gate="G$1" pin="2"/>
-</segment>
 <segment>
 <pinref part="P+3" gate="VCC" pin="VCC"/>
@@
 </segment>
 </net>
-<net name="N$5" class="0">
-<segment>
-<pinref part="Q1" gate="G$1" pin="D"/>
-<wire x1="88.9" y1="33.02" x2="86.36" y2="33.02" width="0.1524" layer="91"/>
-<wire x1="86.36" y1="33.02" x2="86.36" y2="30.48" width="0.1524" layer="91"/>
-<pinref part="SP1" gate="G$1" pin="1"/>
-<wire x1="86.36" y1="30.48" x2="81.28" y2="30.48" width="0.1524" layer="91"/>
-</segment>
-</net>
