File: Esquemático_Sem_Módulo_SD/Schematic_without_SD_Card.brd (EAGLE design)
At the start: 65.7 x 48.2 mm, 8 parts

Commit message: Melhorei a placa de processamento
Parts:
- removed U$4: SWITCH_3PIN, CRD:SWITCH_3PIN
- added U$3: PRESSION_BUTTON, CRD:PRESSION_BUTTON_FOOTPRINT
- moved U$6 18.1 mm to (53.4, 47.8), turned to 180 degrees
- moved R1 9.22 mm to (55.9, 29.9)
- moved LED1 8.24 mm to (54.9, 39.6), turned to 180 degrees
- moved U$2 0.74 mm to (8.78, 28.3)
- moved U$5 0.66 mm to (53.4, 55.3), turned to 180 degrees
- moved ARDUINO_NANO1 0.49 mm to (29.2, 50.0)
- flipped U$1 to the bottom
Connections:
- removed net N$12: ARDUINO_NANO1.19, U$6.2
- removed net N$15: U$4.2, U$6.1
- new net N$4: ARDUINO_NANO1.15, U$3.PL3, U$3.PR3
- net GND: now also ARDUINO_NANO1.19, U$6.2
- net VCC: now also U$3.PL2, U$3.PR2, U$6.1; no longer ARDUINO_NANO1.15, U$4.3
Routing:
- net GND: track 138.6 -> 0.07 mm
- net N$12: track 41.6 -> 0.00 mm
- net N$11: track 37.2 -> 48.8 mm
- net N$1: track 29.6 -> 19.6 mm
- net N$2: track 90.2 -> 80.5 mm
- net N$15: track 8.22 -> 0.00 mm
- net VCC: track 26.4 -> 18.7 mm
- net N$5: track 39.9 -> 41.1 mm
- net N$10: track 4.64 -> 5.51 mm
- net N$3: track 70.2 -> 70.9 mm
- added copper zone on layer 16, net GND
Other:
- board size 65.7 x 48.2 mm -> 64.7 x 48.2 mm
