File: Esquemático_Sem_Módulo_SD/Schematic_without_SD_Card.sch (EAGLE design)
At the start: 8 parts

Commit message: Melhorei a placa de processamento
Parts:
- removed U$4: SWITCH_3PIN, CRD:SWITCH_3PIN
- added U$3: PRESSION_BUTTON, CRD:PRESSION_BUTTON
Connections:
- removed net N$12: ARDUINO_NANO1.GND@1, U$6.2
- removed net N$15: U$4.2, U$6.1
- new net N$4: ARDUINO_NANO1.VIN, U$3.PL3, U$3.PR3
- net GND: now also ARDUINO_NANO1.GND@1, U$6.2
- net VCC: now also U$3.PL2, U$3.PR2, U$6.1; no longer ARDUINO_NANO1.VIN, U$4.3
Changed lines of the file:
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@@
 <drawing>
 <settings>
-<setting alwaysvectorfont="no"/>
+<setting alwaysvectorfont="yes"/>
 <setting verticaltext="up"/>
 </settings>
@@
 <part name="LED1" library="led" library_urn="urn:adsk.eagle:library:259" deviceset="LED" device="5MM" package3d_urn="urn:adsk.eagle:package:15799/2"/>
 <part name="R1" library="rcl" library_urn="urn:adsk.eagle:library:334" deviceset="R-EU_" device="0207/10" package3d_urn="urn:adsk.eagle:package:23491/2"/>
-<part name="U$4" library="CRD" library_urn="urn:adsk.eagle:library:39051337" deviceset="SWITCH_3PIN" device="" package3d_urn="urn:adsk.eagle:package:39192263/6"/>
 <part name="U$5" library="CRD" library_urn="urn:adsk.eagle:library:39051337" deviceset="JST2.54X2P" device="" package3d_urn="urn:adsk.eagle:package:39191967/2"/>
 <part name="U$6" library="CRD" library_urn="urn:adsk.eagle:library:39051337" deviceset="JST2.54X2P" device="" package3d_urn="urn:adsk.eagle:package:39191967/2"/>
+<part name="U$3" library="CRD" library_urn="urn:adsk.eagle:library:39051337" deviceset="PRESSION_BUTTON" device=""/>
 </parts>
 <sheets>
@@
 <attribute name="VALUE" x="201.422" y="120.65" size="1.778" layer="96" rot="R90"/>
 </instance>
-<instance part="U$4" gate="G$1" x="68.58" y="66.04" smashed="yes"/>
 <instance part="U$5" gate="G$1" x="71.12" y="132.08" smashed="yes"/>
 <instance part="U$6" gate="G$1" x="48.26" y="132.08" smashed="yes"/>
+<instance part="U$3" gate="G$1" x="60.96" y="96.52" smashed="yes"/>
 </instances>
 <busses>
@@
 <wire x1="198.12" y1="114.3" x2="147.32" y2="114.3" width="0.1524" layer="91"/>
 </segment>
+<segment>
+<pinref part="U$6" gate="G$1" pin="2"/>
+<wire x1="50.8" y1="121.92" x2="50.8" y2="119.38" width="0.1524" layer="91"/>
+<wire x1="50.8" y1="119.38" x2="101.6" y2="119.38" width="0.1524" layer="91"/>
+<wire x1="101.6" y1="119.38" x2="101.6" y2="109.22" width="0.1524" layer="91"/>
+<pinref part="ARDUINO_NANO1" gate="G$1" pin="GND@1"/>
+<wire x1="101.6" y1="109.22" x2="104.14" y2="109.22" width="0.1524" layer="91"/>
+<label x="101.6" y="121.92" size="1.778" layer="95"/>
+</segment>
 </net>
 <net name="N$5" class="0">
@@
 </segment>
 </net>
-<net name="N$12" class="0">
-<segment>
-<pinref part="U$6" gate="G$1" pin="2"/>
-<wire x1="50.8" y1="121.92" x2="50.8" y2="119.38" width="0.1524" layer="91"/>
-<wire x1="50.8" y1="119.38" x2="101.6" y2="119.38" width="0.1524" layer="91"/>
-<wire x1="101.6" y1="119.38" x2="101.6" y2="109.22" width="0.1524" layer="91"/>
-<pinref part="ARDUINO_NANO1" gate="G$1" pin="GND@1"/>
-<wire x1="101.6" y1="109.22" x2="104.14" y2="109.22" width="0.1524" layer="91"/>
-</segment>
-</net>
 <net name="N$13" class="0">
 <segment>
@@
 <net name="VCC" class="0">
 <segment>
-<pinref part="U$4" gate="G$1" pin="3"/>
-<wire x1="73.66" y1="53.34" x2="139.7" y2="53.34" width="0.1524" layer="91"/>
+<pinref part="U$6" gate="G$1" pin="1"/>
+<wire x1="45.72" y1="121.92" x2="25.4" y2="121.92" width="0.1524" layer="91"/>
+<wire x1="25.4" y1="121.92" x2="25.4" y2="48.26" width="0.1524" layer="91"/>
+<wire x1="25.4" y1="48.26" x2="53.34" y2="48.26" width="0.1524" layer="91"/>
+<wire x1="53.34" y1="48.26" x2="53.34" y2="83.82" width="0.1524" layer="91"/>
+<wire x1="53.34" y1="83.82" x2="68.834" y2="83.82" width="0.1524" layer="91"/>
+<pinref part="U$3" gate="G$1" pin="PL2"/>
+<wire x1="68.834" y1="83.82" x2="68.834" y2="87.63" width="0.1524" layer="91"/>
+<pinref part="U$3" gate="G$1" pin="PR2"/>
+<wire x1="71.374" y1="105.41" x2="71.12" y2="105.41" width="0.1524" layer="91"/>
+<wire x1="71.12" y1="105.41" x2="71.12" y2="111.76" width="0.1524" layer="91"/>
+<wire x1="71.12" y1="111.76" x2="43.18" y2="111.76" width="0.1524" layer="91"/>
+<wire x1="43.18" y1="111.76" x2="43.18" y2="86.36" width="0.1524" layer="91"/>
+<wire x1="43.18" y1="86.36" x2="53.34" y2="86.36" width="0.1524" layer="91"/>
+<wire x1="53.34" y1="86.36" x2="53.34" y2="83.82" width="0.1524" layer="91"/>
+<junction x="53.34" y="83.82"/>
+</segment>
+</net>
+<net name="N$4" class="0">
+<segment>
+<pinref part="ARDUINO_NANO1" gate="G$1" pin="VIN"/>
+<pinref part="U$3" gate="G$1" pin="PR3"/>
+<wire x1="76.454" y1="105.41" x2="76.2" y2="105.41" width="0.1524" layer="91"/>
+<wire x1="76.2" y1="105.41" x2="76.2" y2="111.76" width="0.1524" layer="91"/>
+<wire x1="83.82" y1="111.76" x2="76.2" y2="111.76" width="0.1524" layer="91"/>
+<pinref part="U$3" gate="G$1" pin="PL3"/>
+<wire x1="73.914" y1="86.36" x2="73.914" y2="87.63" width="0.1524" layer="91"/>
+<wire x1="83.82" y1="86.36" x2="73.914" y2="86.36" width="0.1524" layer="91"/>
+<wire x1="83.82" y1="86.36" x2="83.82" y2="111.76" width="0.1524" layer="91"/>
+<junction x="83.82" y="86.36"/>
+<wire x1="83.82" y1="53.34" x2="83.82" y2="86.36" width="0.1524" layer="91"/>
+<wire x1="83.82" y1="53.34" x2="139.7" y2="53.34" width="0.1524" layer="91"/>
 <wire x1="139.7" y1="53.34" x2="139.7" y2="73.66" width="0.1524" layer="91"/>
 <wire x1="139.7" y1="73.66" x2="154.94" y2="73.66" width="0.1524" layer="91"/>
@@
 <wire x1="154.94" y1="91.44" x2="149.86" y2="91.44" width="0.1524" layer="91"/>
 <wire x1="149.86" y1="91.44" x2="149.86" y2="116.84" width="0.1524" layer="91"/>
-<pinref part="ARDUINO_NANO1" gate="G$1" pin="VIN"/>
 <wire x1="149.86" y1="116.84" x2="144.78" y2="116.84" width="0.1524" layer="91"/>
 </segment>
 </net>
-<net name="N$15" class="0">
-<segment>
-<pinref part="U$6" gate="G$1" pin="1"/>
-<wire x1="45.72" y1="121.92" x2="25.4" y2="121.92" width="0.1524" layer="91"/>
-<wire x1="25.4" y1="121.92" x2="25.4" y2="48.26" width="0.1524" layer="91"/>
-<wire x1="25.4" y1="48.26" x2="68.58" y2="48.26" width="0.1524" layer="91"/>
-<pinref part="U$4" gate="G$1" pin="2"/>
-<wire x1="68.58" y1="48.26" x2="68.58" y2="53.34" width="0.1524" layer="91"/>
-</segment>
-</net>
