File: Esquemático acionamento/versão 01 acionamento/Esquemático.brd (EAGLE design)
At the start: 24.1 x 47.9 mm, 7 parts, among them Q2 IRF540

Commit message: Modificação
Routing:
- net VCC: track 23.3 -> 24.4 mm
Changed lines of the file:
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@@
 <drawing>
 <settings>
-<setting alwaysvectorfont="no"/>
+<setting alwaysvectorfont="yes"/>
 <setting verticaltext="up"/>
 </settings>
@@
 <param name="msMicroVia" value="9.99mm"/>
 <param name="msBlindViaRatio" value="0.5"/>
-<param name="rvPadTop" value="0.25"/>
+<param name="rvPadTop" value="0.5"/>
 <param name="rvPadInner" value="0.25"/>
-<param name="rvPadBottom" value="0.25"/>
+<param name="rvPadBottom" value="0.5"/>
 <param name="rvViaOuter" value="0.25"/>
 <param name="rvViaInner" value="0.25"/>
@@
 <param name="rvMicroViaInner" value="0.25"/>
 <param name="rlMinPadTop" value="10mil"/>
-<param name="rlMaxPadTop" value="20mil"/>
+<param name="rlMaxPadTop" value="30mil"/>
 <param name="rlMinPadInner" value="10mil"/>
 <param name="rlMaxPadInner" value="20mil"/>
 <param name="rlMinPadBottom" value="10mil"/>
-<param name="rlMaxPadBottom" value="20mil"/>
+<param name="rlMaxPadBottom" value="30mil"/>
 <param name="rlMinViaOuter" value="8mil"/>
 <param name="rlMaxViaOuter" value="20mil"/>
@@
 </autorouter>
 <elements>
-<element name="Q2" library="transistor-fet" library_urn="urn:adsk.eagle:library:396" package="TO220" package3d_urn="urn:adsk.eagle:package:28520/1" value="IRF540" x="-15.24" y="-10.922" smashed="yes">
+<element name="Q2" library="transistor-fet" library_urn="urn:adsk.eagle:library:43498060" package="TO220" package3d_urn="urn:adsk.eagle:package:43498084/1" value="IRF540" x="-15.24" y="-10.922" smashed="yes">
 <attribute name="NAME" x="-19.05" y="-5.715" size="1.778" layer="25" ratio="10"/>
 <attribute name="POPULARITY" value="5" x="15.24" y="-19.812" size="1.778" layer="27" display="off"/>
@@
 <contactref element="R1" pad="2"/>
 <contactref element="Q2" pad="1"/>
-<wire x1="-17.78" y1="-24.13" x2="-17.78" y2="-17.272" width="1" layer="16"/>
-<wire x1="-17.78" y1="-17.272" x2="-25.4" y2="-24.892" width="1" layer="16"/>
-<wire x1="-25.4" y1="-24.892" x2="-25.4" y2="-29.21" width="1" layer="16"/>
+<wire x1="-17.78" y1="-24.13" x2="-17.78" y2="-17.272" width="1.5" layer="16"/>
+<wire x1="-17.78" y1="-17.272" x2="-25.4" y2="-24.892" width="1.5" layer="16"/>
+<wire x1="-25.4" y1="-24.892" x2="-25.4" y2="-29.21" width="1.5" layer="16"/>
 </signal>
 <signal name="VCC">
 <contactref element="U$3" pad="1"/>
 <contactref element="U$2" pad="1"/>
-<wire x1="-27.94" y1="-2.286" x2="-25.527" y2="0.127" width="1" layer="16"/>
-<wire x1="-25.4" y1="-9.652" x2="-27.94" y2="-12.192" width="1" layer="16"/>
-<wire x1="-27.94" y1="-12.192" x2="-27.94" y2="-16.51" width="1" layer="16"/>
+<wire x1="-26.416" y1="0.127" x2="-25.527" y2="0.127" width="1.5" layer="16"/>
+<wire x1="-26.416" y1="0.127" x2="-27.94" y2="-1.397" width="1.5" layer="16"/>
+<wire x1="-25.4" y1="-9.652" x2="-26.289" y2="-9.652" width="1.5" layer="16"/>
+<wire x1="-26.289" y1="-9.652" x2="-27.94" y2="-11.303" width="1.5" layer="16"/>
+<wire x1="-27.94" y1="-11.303" x2="-27.94" y2="-16.51" width="1.5" layer="16"/>
 <contactref element="U$4" pad="2"/>
-<wire x1="-25.4" y1="-19.05" x2="-27.94" y2="-16.51" width="1" layer="16"/>
-<wire x1="-25.4" y1="-9.652" x2="-27.94" y2="-7.112" width="1" layer="16"/>
-<wire x1="-27.94" y1="-7.112" x2="-27.94" y2="-2.286" width="1" layer="16"/>
+<wire x1="-25.4" y1="-19.05" x2="-27.94" y2="-16.51" width="1.5" layer="16"/>
+<wire x1="-25.4" y1="-9.652" x2="-27.94" y2="-7.112" width="1.5" layer="16"/>
+<wire x1="-27.94" y1="-7.112" x2="-27.94" y2="-1.397" width="1.5" layer="16"/>
 </signal>
 <signal name="GND">
@@
 <contactref element="U$1" pad="2"/>
 <contactref element="SP1" pad="+"/>
-<wire x1="-16.256" y1="-31.75" x2="-25.4" y2="-31.75" width="1" layer="16"/>
+<wire x1="-16.256" y1="-31.75" x2="-25.4" y2="-31.75" width="1.5" layer="16"/>
 </signal>
 <signal name="DRENO">
@@
 <contactref element="U$2" pad="2"/>
 <contactref element="Q2" pad="2"/>
-<wire x1="-17.145" y1="-9.525" x2="-24.257" y2="-2.413" width="1" layer="16"/>
-<wire x1="-25.527" y1="-2.413" x2="-24.257" y2="-2.413" width="1" layer="16"/>
-<wire x1="-17.145" y1="-9.525" x2="-15.24" y2="-11.43" width="1" layer="16"/>
-<wire x1="-15.24" y1="-11.43" x2="-15.24" y2="-17.272" width="1" layer="16"/>
-<wire x1="-25.4" y1="-12.192" x2="-21.336" y2="-12.192" width="1" layer="16"/>
-<wire x1="-17.145" y1="-9.525" x2="-18.669" y2="-9.525" width="1" layer="16"/>
-<wire x1="-18.669" y1="-9.525" x2="-21.336" y2="-12.192" width="1" layer="16"/>
+<wire x1="-17.145" y1="-9.525" x2="-24.257" y2="-2.413" width="1.5" layer="16"/>
+<wire x1="-25.527" y1="-2.413" x2="-24.257" y2="-2.413" width="1.5" layer="16"/>
+<wire x1="-17.145" y1="-9.525" x2="-15.24" y2="-11.43" width="1.5" layer="16"/>
+<wire x1="-15.24" y1="-11.43" x2="-15.24" y2="-17.272" width="1.5" layer="16"/>
+<wire x1="-25.4" y1="-12.192" x2="-21.336" y2="-12.192" width="1.5" layer="16"/>
+<wire x1="-17.145" y1="-9.525" x2="-18.669" y2="-9.525" width="1.5" layer="16"/>
+<wire x1="-18.669" y1="-9.525" x2="-21.336" y2="-12.192" width="1.5" layer="16"/>
 </signal>
 </signals>
