File: Esquemático acionamento/versão 01 acionamento/Esquemático.brd (EAGLE design)
At the start: 24.1 x 47.9 mm, 7 parts, among them Q2 IRF540

Commit message: Update
Routing:
- net DRENO: track 29.2 -> 27.2 mm
Changed lines of the file:
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@@
 <grid distance="100" unitdist="mil" unit="mm" style="lines" multiple="1" display="yes" altdistance="5" altunitdist="mil" altunit="mm"/>
 <layers>
-<layer number="1" name="Top" color="4" fill="1" visible="no" active="yes"/>
+<layer number="1" name="Top" color="4" fill="1" visible="yes" active="yes"/>
 <layer number="2" name="Route2" color="16" fill="1" visible="no" active="no"/>
 <layer number="3" name="Route3" color="17" fill="1" visible="no" active="no"/>
@@
 <hole x="-27.94" y="5.08" drill="3"/>
 <hole x="-8.89" y="5.207" drill="3"/>
-<dimension x1="-30.46" y1="-40.31" x2="-6.35" y2="-40.31" x3="-18.405" y3="-45.72" textsize="1.778" layer="16"/>
-<dimension x1="-6.35" y1="7.62" x2="-6.858" y2="-40.386" x3="10.16" y3="-16.383" textsize="1.778" layer="16" dtype="vertical"/>
 </plain>
 <attributes>
@@
 </class>
 </classes>
-<designrules name="default *">
+<designrules name="default">
 <description language="de">&lt;b&gt;EAGLE Design Rules&lt;/b&gt;
 &lt;p&gt;
@@
 <param name="mtCopper" value="0.035mm 0.035mm 0.035mm 0.035mm 0.035mm 0.035mm 0.035mm 0.035mm 0.035mm 0.035mm 0.035mm 0.035mm 0.035mm 0.035mm 0.035mm 0.035mm"/>
 <param name="mtIsolate" value="1.5mm 0.15mm 0.2mm 0.15mm 0.2mm 0.15mm 0.2mm 0.15mm 0.2mm 0.15mm 0.2mm 0.15mm 0.2mm 0.15mm 0.2mm"/>
-<param name="mdWireWire" value="20mil"/>
+<param name="mdWireWire" value="30mil"/>
 <param name="mdWirePad" value="20mil"/>
 <param name="mdWireVia" value="20mil"/>
@@
 <param name="mdDrill" value="6mil"/>
 <param name="mdSmdStop" value="0mil"/>
-<param name="msWidth" value="1mm"/>
+<param name="msWidth" value="1.5mm"/>
 <param name="msDrill" value="0.35mm"/>
 <param name="msMicroVia" value="9.99mm"/>
 <param name="msBlindViaRatio" value="0.5"/>
-<param name="rvPadTop" value="0.5"/>
+<param name="rvPadTop" value="0.35"/>
 <param name="rvPadInner" value="0.25"/>
-<param name="rvPadBottom" value="0.5"/>
+<param name="rvPadBottom" value="0.35"/>
 <param name="rvViaOuter" value="0.25"/>
 <param name="rvViaInner" value="0.25"/>
@@
 <contactref element="U$2" pad="2"/>
 <contactref element="Q2" pad="2"/>
-<wire x1="-17.145" y1="-9.525" x2="-24.257" y2="-2.413" width="1.5" layer="16"/>
-<wire x1="-25.527" y1="-2.413" x2="-24.257" y2="-2.413" width="1.5" layer="16"/>
-<wire x1="-17.145" y1="-9.525" x2="-15.24" y2="-11.43" width="1.5" layer="16"/>
-<wire x1="-15.24" y1="-11.43" x2="-15.24" y2="-17.272" width="1.5" layer="16"/>
 <wire x1="-25.4" y1="-12.192" x2="-21.336" y2="-12.192" width="1.5" layer="16"/>
-<wire x1="-17.145" y1="-9.525" x2="-18.669" y2="-9.525" width="1.5" layer="16"/>
+<wire x1="-18.669" y1="-9.525" x2="-18.415" y2="-9.525" width="1.5" layer="16"/>
 <wire x1="-18.669" y1="-9.525" x2="-21.336" y2="-12.192" width="1.5" layer="16"/>
+<wire x1="-15.24" y1="-12.7" x2="-15.24" y2="-17.272" width="1.5" layer="16"/>
+<wire x1="-18.415" y1="-9.525" x2="-25.527" y2="-2.413" width="1.5" layer="16"/>
+<wire x1="-18.415" y1="-9.525" x2="-15.24" y2="-12.7" width="1.5" layer="16"/>
 </signal>
 </signals>
