File: Esquemático acionamento/versão 02 acionamento/Esquemático.brd (EAGLE design)
At the start: 34.3 x 47.9 mm, 9 parts, among them Q1 IRF540, Q2 IRF540

Commit message: Modificação
Parts:
- moved R2 0.74 mm to (-3.94, -24.1)
- moved R1 0.63 mm to (-14.0, -24.1)
Routing:
- net SKIB: track 32.4 -> 34.2 mm
- net VCC: track 23.3 -> 24.2 mm
