File: Esquemático processamento/Schematic_without_SD_Card.sch (EAGLE design)
At the start: 8 parts

Commit message: Update
Changed lines of the file:
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@@
 <part name="FRAME1" library="frames" library_urn="urn:adsk.eagle:library:229" deviceset="A4L-LOC" device=""/>
 <part name="ARDUINO_NANO1" library="ArduinoNanoV30" library_urn="urn:adsk.eagle:library:39315983" deviceset="ARDUINO_NANO" device="" package3d_urn="urn:adsk.eagle:package:39315986/2"/>
-<part name="U$1" library="CRD" library_urn="urn:adsk.eagle:library:39051337" deviceset="BMP280" device="V1" package3d_urn="urn:adsk.eagle:package:39029072/5"/>
-<part name="U$2" library="CRD" library_urn="urn:adsk.eagle:library:39051337" deviceset="MPU6050" device="V1" package3d_urn="urn:adsk.eagle:package:39029071/7"/>
+<part name="U$1" library="CRD" library_urn="urn:adsk.eagle:library:39051337" deviceset="BMP280" device="V1" package3d_urn="urn:adsk.eagle:package:39029072/6"/>
+<part name="U$2" library="CRD" library_urn="urn:adsk.eagle:library:39051337" deviceset="MPU6050" device="V1" package3d_urn="urn:adsk.eagle:package:39029071/8"/>
 <part name="LED1" library="led" library_urn="urn:adsk.eagle:library:259" deviceset="LED" device="5MM" package3d_urn="urn:adsk.eagle:package:15799/2"/>
 <part name="R1" library="rcl" library_urn="urn:adsk.eagle:library:334" deviceset="R-EU_" device="0207/10" package3d_urn="urn:adsk.eagle:package:23491/2"/>
 <part name="U$5" library="CRD" library_urn="urn:adsk.eagle:library:39051337" deviceset="JST2.54X2P" device="" package3d_urn="urn:adsk.eagle:package:39191967/2"/>
 <part name="U$6" library="CRD" library_urn="urn:adsk.eagle:library:39051337" deviceset="JST2.54X2P" device="" package3d_urn="urn:adsk.eagle:package:39191967/2"/>
-<part name="U$3" library="CRD" library_urn="urn:adsk.eagle:library:39051337" deviceset="PRESSION_BUTTON" device="" package3d_urn="urn:adsk.eagle:package:43483815/2"/>
+<part name="U$3" library="CRD" library_urn="urn:adsk.eagle:library:39051337" deviceset="PRESSION_BUTTON" device="" package3d_urn="urn:adsk.eagle:package:43483815/3"/>
 </parts>
 <sheets>
@@
 <wire x1="25.4" y1="48.26" x2="53.34" y2="48.26" width="0.1524" layer="91"/>
 <wire x1="53.34" y1="48.26" x2="53.34" y2="83.82" width="0.1524" layer="91"/>
-<wire x1="53.34" y1="83.82" x2="68.834" y2="83.82" width="0.1524" layer="91"/>
+<wire x1="53.34" y1="83.82" x2="69.85" y2="83.82" width="0.1524" layer="91"/>
 <pinref part="U$3" gate="G$1" pin="PL2"/>
-<wire x1="68.834" y1="83.82" x2="68.834" y2="87.63" width="0.1524" layer="91"/>
 <pinref part="U$3" gate="G$1" pin="PR2"/>
-<wire x1="71.374" y1="105.41" x2="71.12" y2="105.41" width="0.1524" layer="91"/>
+<wire x1="69.85" y1="109.22" x2="71.12" y2="105.41" width="0.1524" layer="91"/>
 <wire x1="71.12" y1="105.41" x2="71.12" y2="111.76" width="0.1524" layer="91"/>
 <wire x1="71.12" y1="111.76" x2="43.18" y2="111.76" width="0.1524" layer="91"/>
@@
 <pinref part="ARDUINO_NANO1" gate="G$1" pin="VIN"/>
 <pinref part="U$3" gate="G$1" pin="PR3"/>
-<wire x1="76.454" y1="105.41" x2="76.2" y2="105.41" width="0.1524" layer="91"/>
+<wire x1="74.93" y1="109.22" x2="76.2" y2="105.41" width="0.1524" layer="91"/>
 <wire x1="76.2" y1="105.41" x2="76.2" y2="111.76" width="0.1524" layer="91"/>
 <wire x1="83.82" y1="111.76" x2="76.2" y2="111.76" width="0.1524" layer="91"/>
 <pinref part="U$3" gate="G$1" pin="PL3"/>
-<wire x1="73.914" y1="86.36" x2="73.914" y2="87.63" width="0.1524" layer="91"/>
+<wire x1="73.914" y1="86.36" x2="74.93" y2="83.82" width="0.1524" layer="91"/>
 <wire x1="83.82" y1="86.36" x2="73.914" y2="86.36" width="0.1524" layer="91"/>
 <wire x1="83.82" y1="86.36" x2="83.82" y2="111.76" width="0.1524" layer="91"/>
