File: Esquemático processamento/Schematic_without_SD_Card.brd (EAGLE design)
At the start: 64.7 x 48.2 mm, 8 parts

Commit message: Update
Parts:
- moved U$3 12.4 mm to (45.1, 28.1)
Routing:
- net GND: track 93.7 -> 47.4 mm
- net VCC: track 23.1 -> 0.00 mm
- net N$4: track 16.4 -> 0.00 mm
Changed lines of the file:
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@@
 </layers>
 <board>
-<fusionsync huburn="a.YnVzaW5lc3M6Z21haWwzOTY3MDkw" projecturn="a.YnVzaW5lc3M6Z21haWwzOTY3MDkwI0QyMDI0MDIyMjczNjgyMTMwMQ" f3durn="urn:adsk.wipprod:dm.lineage:4HcadxyTRMiACPfFyTq5TQ" pcbguid="" lastpulledtime="" lastsyncedchangeguid="" latestrevisionid="69e20167-c29c-4609-bc9a-65bf308ef2df" lastsyncedrevisionid="69e20167-c29c-4609-bc9a-65bf308ef2df" lastboardhashguid="7a9dff24-2713-eebe-dc70-94a094832090" lastpushedtime="2024-02-28T02:08:44Z" linktopcb3d="false"/>
+<fusionsync huburn="a.YnVzaW5lc3M6ZGlzY2VudGUxNzg" projecturn="a.YnVzaW5lc3M6ZGlzY2VudGUxNzgjRDIwMjIwNjExNTMyNjQzNTAx" f3durn="urn:adsk.wipprod:dm.lineage:tcO9UwKJQUiMCS_hZ89ZqA" pcbguid="" lastpulledtime="" lastsyncedchangeguid="" latestrevisionid="acf1e47a-85b1-45ab-9a50-db8dbe08f255" lastsyncedrevisionid="acf1e47a-85b1-45ab-9a50-db8dbe08f255" lastboardhashguid="134e2b11-63d4-36dc-5cf1-f8650a257b7e" lastpushedtime="2024-03-04T15:19:45Z" linktopcb3d="true"/>
 <plain>
 <wire x1="-3.81" y1="16.51" x2="60.9" y2="16.51" width="0" layer="20"/>
@@
 <attribute name="VALUE" x="56.515" y="27.6494" size="1.27" layer="27" ratio="10" rot="R90"/>
 </element>
-<element name="U$1" library="CRD" library_urn="urn:adsk.eagle:library:39051337" package="BMP280_FOOTPRINT" package3d_urn="urn:adsk.eagle:package:39029072/5" value="BMP280V1" x="30.02" y="27.67" smashed="yes" rot="MR180"/>
-<element name="U$2" library="CRD" library_urn="urn:adsk.eagle:library:39051337" package="MPU6050_FOOTPRINT" package3d_urn="urn:adsk.eagle:package:39029071/7" value="MPU6050V1" x="8.779" y="28.305" smashed="yes" rot="R90"/>
+<element name="U$1" library="CRD" library_urn="urn:adsk.eagle:library:39051337" package="BMP280_FOOTPRINT" package3d_urn="urn:adsk.eagle:package:39029072/6" value="BMP280V1" x="30.02" y="27.67" smashed="yes" rot="MR180"/>
+<element name="U$2" library="CRD" library_urn="urn:adsk.eagle:library:39051337" package="MPU6050_FOOTPRINT" package3d_urn="urn:adsk.eagle:package:39029071/8" value="MPU6050V1" x="8.779" y="28.305" smashed="yes" rot="R90"/>
 <element name="U$5" library="CRD" library_urn="urn:adsk.eagle:library:39051337" package="JST2.54X2P_FOOTPRINT" package3d_urn="urn:adsk.eagle:package:39191967/2" value="JST2.54X2P" x="53.39" y="55.31" smashed="yes" rot="R180"/>
 <element name="U$6" library="CRD" library_urn="urn:adsk.eagle:library:39051337" package="JST2.54X2P_FOOTPRINT" package3d_urn="urn:adsk.eagle:package:39191967/2" value="JST2.54X2P" x="53.422" y="47.774" smashed="yes" rot="R180"/>
-<element name="U$3" library="CRD" library_urn="urn:adsk.eagle:library:39051337" package="PRESSION_BUTTON_FOOTPRINT" package3d_urn="urn:adsk.eagle:package:43483815/2" value="PRESSION_BUTTON" x="42.1114" y="40.078796875" smashed="yes" rot="R270"/>
+<element name="U$3" library="CRD" library_urn="urn:adsk.eagle:library:39051337" package="PRESSION_BUTTON_FOOTPRINT" package3d_urn="urn:adsk.eagle:package:43483815/3" value="PRESSION_BUTTON" x="45.1114" y="28.078796875" smashed="yes" rot="R270"/>
 </elements>
 <signals>
@@
 <contactref element="U$6" pad="2"/>
 <contactref element="ARDUINO_NANO1" pad="19"/>
-<wire x1="36.83" y1="57.642" x2="36.83" y2="55.17" width="1.5" layer="16"/>
-<wire x1="36.83" y1="55.17" x2="42" y2="50" width="1.5" layer="16"/>
-<wire x1="42" y1="50" x2="42" y2="42.492" width="1.5" layer="16"/>
-<wire x1="42" y1="42.492" x2="41.91" y2="42.402" width="1.5" layer="16"/>
 <wire x1="19.006" y1="22.033" x2="22.30443125" y2="22.033" width="1.5" layer="1"/>
 <wire x1="19.006" y1="22.033" x2="18.9635" y2="21.9905" width="1.5" layer="1"/>
@@
 <wire x1="25.135715625" y1="24.864284375" x2="26.0855" y2="25.81406875" width="1.5" layer="1"/>
 <wire x1="25.17" y1="24.83" x2="25.135715625" y2="24.864284375" width="1.5" layer="1"/>
-<wire x1="55.88" y1="24.83" x2="42" y2="24.83" width="1.5" layer="1"/>
-<wire x1="42" y1="24.83" x2="41.746" y2="24.83" width="1.5" layer="1"/>
-<wire x1="41.746" y1="24.83" x2="25.17" y2="24.83" width="1.5" layer="1"/>
-<wire x1="41.91" y1="24.92" x2="42" y2="24.83" width="1.5" layer="1"/>
-<wire x1="41.91" y1="42.402" x2="41.746" y2="42.238" width="1.5" layer="1"/>
-<wire x1="41.746" y1="42.238" x2="41.746" y2="24.83" width="1.5" layer="1"/>
-<wire x1="52.152" y1="47.774" x2="44.226" y2="47.774" width="1.5" layer="16"/>
-<wire x1="44.226" y1="47.774" x2="42" y2="50" width="1.5" layer="16"/>
+<wire x1="55.88" y1="24.83" x2="40" y2="24.83" width="1.5" layer="1"/>
+<wire x1="25.17" y1="24.83" x2="40" y2="24.83" width="1.5" layer="1"/>
+<wire x1="41.91" y1="42.402" x2="52.152" y2="47.774" width="0" layer="19" extent="1-1"/>
+<wire x1="36.83" y1="57.642" x2="41.91" y2="42.402" width="0" layer="19" extent="1-1"/>
+<wire x1="26.0855" y1="33.79" x2="41.91" y2="42.402" width="0" layer="19" extent="1-1"/>
 </signal>
 <signal name="N$5">
@@
 <contactref element="U$2" pad="VCC"/>
 <wire x1="18.9635" y1="19.3905" x2="32.4405" y2="19.3905" width="1.5" layer="16"/>
-<wire x1="39.18" y1="26.13" x2="32.4405" y2="19.3905" width="1.5" layer="16"/>
-<wire x1="39.18" y1="38.56" x2="36.83" y2="40.91" width="1.5" layer="16"/>
+<wire x1="38.926" y1="25.876" x2="32.4405" y2="19.3905" width="1.5" layer="16"/>
+<wire x1="38.926" y1="38.814" x2="36.83" y2="40.91" width="1.5" layer="16"/>
 <wire x1="36.83" y1="42.402" x2="36.83" y2="40.91" width="1.5" layer="16"/>
-<wire x1="39.18" y1="38.56" x2="39.18" y2="26.13" width="1.5" layer="16"/>
+<wire x1="38.926" y1="38.814" x2="38.926" y2="25.876" width="1.5" layer="16"/>
 </signal>
 <signal name="N$10">
@@
 <contactref element="U$3" pad="PL2"/>
 <contactref element="U$3" pad="PR2"/>
-<wire x1="54.692" y1="47.774" x2="54.652" y2="47.734" width="1.5" layer="16"/>
-<wire x1="54.652" y1="47.734" x2="54.652" y2="46.4844625" width="1.5" layer="16"/>
-<wire x1="54.652" y1="46.4844625" x2="53.1675375" y2="45" width="1.5" layer="16"/>
-<wire x1="53.1675375" y1="45" x2="51" y2="45" width="1.5" layer="16"/>
-<wire x1="51" y1="45" x2="50" y2="44" width="1.5" layer="16"/>
-<wire x1="50" y1="44" x2="50" y2="33.82" width="1.5" layer="16"/>
-<wire x1="46.6114" y1="33.878796875" x2="49.941203125" y2="33.878796875" width="1.5" layer="16"/>
-<wire x1="49.941203125" y1="33.878796875" x2="50" y2="33.82" width="1.5" layer="16"/>
-<wire x1="44.1114" y1="33.878796875" x2="46.6114" y2="33.878796875" width="1.5" layer="16"/>
+<wire x1="46.3094" y1="32.881796875" x2="54.692" y2="47.774" width="0" layer="19" extent="1-1"/>
+<wire x1="43.8094" y1="32.881796875" x2="46.3094" y2="32.881796875" width="0" layer="19" extent="1-1"/>
 </signal>
 <signal name="N$4">
@@
 <contactref element="U$3" pad="PL3"/>
 <contactref element="U$3" pad="PR3"/>
-<wire x1="46.6114" y1="31.178796875" x2="44.1114" y2="31.178796875" width="1.5" layer="16"/>
-<wire x1="44.45" y1="42.402" x2="44.45" y2="41.323" width="1.5" layer="16"/>
-<wire x1="41.746" y1="32.492" x2="43.059203125" y2="31.178796875" width="1.5" layer="16"/>
-<wire x1="43.059203125" y1="31.178796875" x2="44.1114" y2="31.178796875" width="1.5" layer="16"/>
-<wire x1="44.45" y1="41.323" x2="41.746" y2="38.619" width="1.5" layer="16"/>
-<wire x1="41.746" y1="38.619" x2="41.746" y2="32.492" width="1.5" layer="16"/>
+<wire x1="46.3094" y1="29.881796875" x2="44.45" y2="42.402" width="0" layer="19" extent="1-1"/>
+<wire x1="43.8094" y1="29.881796875" x2="46.3094" y2="29.881796875" width="0" layer="19" extent="1-1"/>
 </signal>
 </signals>

Commit message: Update
Connections:
- net N$2: now also U$1.SDO
- net N$3: now also U$1.CSB
- net VCC: now also U$3.PL1
Changed lines of the file:
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@@
 <layers>
 <layer number="1" name="Top" color="4" fill="1" visible="yes" active="yes"/>
-<layer number="2" name="Route2" color="16" fill="1" visible="no" active="yes"/>
-<layer number="3" name="Route3" color="17" fill="1" visible="no" active="yes"/>
-<layer number="4" name="Route4" color="18" fill="1" visible="no" active="yes"/>
-<layer number="5" name="Route5" color="19" fill="1" visible="no" active="yes"/>
-<layer number="6" name="Route6" color="25" fill="1" visible="no" active="yes"/>
-<layer number="7" name="Route7" color="26" fill="1" visible="no" active="yes"/>
-<layer number="8" name="Route8" color="27" fill="1" visible="no" active="yes"/>
-<layer number="9" name="Route9" color="28" fill="1" visible="no" active="yes"/>
-<layer number="10" name="Route10" color="29" fill="1" visible="no" active="yes"/>
-<layer number="11" name="Route11" color="30" fill="1" visible="no" active="yes"/>
-<layer number="12" name="Route12" color="20" fill="1" visible="no" active="yes"/>
-<layer number="13" name="Route13" color="21" fill="1" visible="no" active="yes"/>
-<layer number="14" name="Route14" color="22" fill="1" visible="no" active="yes"/>
-<layer number="15" name="Route15" color="23" fill="1" visible="no" active="yes"/>
+<layer number="2" name="Route2" color="16" fill="1" visible="yes" active="yes"/>
+<layer number="3" name="Route3" color="17" fill="1" visible="yes" active="yes"/>
+<layer number="4" name="Route4" color="18" fill="1" visible="yes" active="yes"/>
+<layer number="5" name="Route5" color="19" fill="1" visible="yes" active="yes"/>
+<layer number="6" name="Route6" color="25" fill="1" visible="yes" active="yes"/>
+<layer number="7" name="Route7" color="26" fill="1" visible="yes" active="yes"/>
+<layer number="8" name="Route8" color="27" fill="1" visible="yes" active="yes"/>
+<layer number="9" name="Route9" color="28" fill="1" visible="yes" active="yes"/>
+<layer number="10" name="Route10" color="29" fill="1" visible="yes" active="yes"/>
+<layer number="11" name="Route11" color="30" fill="1" visible="yes" active="yes"/>
+<layer number="12" name="Route12" color="20" fill="1" visible="yes" active="yes"/>
+<layer number="13" name="Route13" color="21" fill="1" visible="yes" active="yes"/>
+<layer number="14" name="Route14" color="22" fill="1" visible="yes" active="yes"/>
+<layer number="15" name="Route15" color="23" fill="1" visible="yes" active="yes"/>
 <layer number="16" name="Bottom" color="1" fill="1" visible="yes" active="yes"/>
 <layer number="17" name="Pads" color="2" fill="1" visible="yes" active="yes"/>
@@
 <layer number="25" name="tNames" color="7" fill="1" visible="yes" active="yes"/>
 <layer number="26" name="bNames" color="7" fill="1" visible="yes" active="yes"/>
-<layer number="27" name="tValues" color="7" fill="1" visible="yes" active="yes"/>
-<layer number="28" name="bValues" color="7" fill="1" visible="yes" active="yes"/>
+<layer number="27" name="tValues" color="7" fill="1" visible="no" active="yes"/>
+<layer number="28" name="bValues" color="7" fill="1" visible="no" active="yes"/>
 <layer number="29" name="tStop" color="7" fill="3" visible="no" active="yes"/>
 <layer number="30" name="bStop" color="7" fill="6" visible="no" active="yes"/>
@@
 <layer number="41" name="tRestrict" color="4" fill="10" visible="yes" active="yes"/>
 <layer number="42" name="bRestrict" color="1" fill="10" visible="yes" active="yes"/>
-<layer number="43" name="vRestrict" color="2" fill="10" visible="yes" active="yes"/>
+<layer number="43" name="vRestrict" color="2" fill="10" visible="no" active="yes"/>
 <layer number="44" name="Drills" color="7" fill="1" visible="no" active="yes"/>
-<layer number="45" name="Holes" color="7" fill="1" visible="yes" active="yes"/>
+<layer number="45" name="Holes" color="7" fill="1" visible="no" active="yes"/>
 <layer number="46" name="Milling" color="3" fill="1" visible="no" active="yes"/>
 <layer number="47" name="Measures" color="7" fill="1" visible="no" active="yes"/>
-<layer number="48" name="Document" color="7" fill="1" visible="yes" active="yes"/>
-<layer number="49" name="Reference" color="7" fill="1" visible="yes" active="yes"/>
+<layer number="48" name="Document" color="7" fill="1" visible="no" active="yes"/>
+<layer number="49" name="Reference" color="7" fill="1" visible="no" active="yes"/>
 <layer number="51" name="tDocu" color="7" fill="1" visible="yes" active="yes"/>
 <layer number="52" name="bDocu" color="7" fill="1" visible="yes" active="yes"/>
@@
 <param name="msMicroVia" value="9.99mm"/>
 <param name="msBlindViaRatio" value="0.5"/>
-<param name="rvPadTop" value="0.8"/>
+<param name="rvPadTop" value="0.25"/>
 <param name="rvPadInner" value="0.25"/>
-<param name="rvPadBottom" value="0.8"/>
+<param name="rvPadBottom" value="0.25"/>
 <param name="rvViaOuter" value="0.25"/>
 <param name="rvViaInner" value="0.25"/>
@@
 <wire x1="26.1905" y1="27.1905" x2="31.1655" y2="32.1655" width="1.5" layer="16"/>
 <wire x1="16.8095" y1="27.1905" x2="18.9635" y2="27.1905" width="1.5" layer="16"/>
+<contactref element="U$1" pad="CSB"/>
+<wire x1="31.1655" y1="33.79" x2="33.7055" y2="33.79" width="0" layer="19" extent="1-1"/>
 </signal>
 <signal name="N$2">
@@
 <wire x1="28.6255" y1="36.6255" x2="28.6255" y2="33.79" width="1.5" layer="16"/>
 <wire x1="29.21" y1="37.21" x2="28.6255" y2="36.6255" width="1.5" layer="16"/>
+<contactref element="U$1" pad="SDO"/>
+<wire x1="28.6255" y1="33.79" x2="36.2455" y2="33.79" width="0" layer="19" extent="1-1"/>
 </signal>
 <signal name="GND">
@@
 <wire x1="55.88" y1="24.83" x2="40" y2="24.83" width="1.5" layer="1"/>
 <wire x1="25.17" y1="24.83" x2="40" y2="24.83" width="1.5" layer="1"/>
-<wire x1="41.91" y1="42.402" x2="52.152" y2="47.774" width="0" layer="19" extent="1-1"/>
-<wire x1="36.83" y1="57.642" x2="41.91" y2="42.402" width="0" layer="19" extent="1-1"/>
-<wire x1="26.0855" y1="33.79" x2="41.91" y2="42.402" width="0" layer="19" extent="1-1"/>
 </signal>
 <signal name="N$5">
@@
 <contactref element="U$3" pad="PL2"/>
 <contactref element="U$3" pad="PR2"/>
-<wire x1="46.3094" y1="32.881796875" x2="54.692" y2="47.774" width="0" layer="19" extent="1-1"/>
-<wire x1="43.8094" y1="32.881796875" x2="46.3094" y2="32.881796875" width="0" layer="19" extent="1-1"/>
+<contactref element="U$3" pad="PL1"/>
+<wire x1="43.8094" y1="35.881796875" x2="54.692" y2="47.774" width="0" layer="19" extent="1-1"/>
+<wire x1="43.8094" y1="32.881796875" x2="43.8094" y2="35.881796875" width="0" layer="19" extent="1-1"/>
+<wire x1="46.3094" y1="32.881796875" x2="43.8094" y2="32.881796875" width="0" layer="19" extent="1-1"/>
 </signal>
 <signal name="N$4">
@@
 <contactref element="U$3" pad="PL3"/>
 <contactref element="U$3" pad="PR3"/>
-<wire x1="46.3094" y1="29.881796875" x2="44.45" y2="42.402" width="0" layer="19" extent="1-1"/>
-<wire x1="43.8094" y1="29.881796875" x2="46.3094" y2="29.881796875" width="0" layer="19" extent="1-1"/>
+<wire x1="43.8094" y1="29.881796875" x2="44.45" y2="42.402" width="0" layer="19" extent="1-1"/>
+<wire x1="46.3094" y1="29.881796875" x2="43.8094" y2="29.881796875" width="0" layer="19" extent="1-1"/>
 </signal>
 </signals>
